File: ffs/ffs.sch (KiCad schematic (older format))
At the start: 33 parts, among them J1 EURO_PWR_2x5, J2 Conn_01x10_Male, U1 4015, U10 4051, U12 4017, U13 4017, U2 4051, U3 4051, U4 4046, U5 4081, U6 4017, U7 4017, U8 4015, U9 4051

Commit message: added button controlled controller, fixed multiplier circuit
Parts:
- added U?: 4081, symbol 4xxx:4081
- J1: symbol eurorack:EURO_PWR_2x5 -> euroraack:EURO_PWR_2x5
Connections:
- net FreqMultOut: now also U5.9, U?.5; no longer U5.6
- net SigIn: now also U?.4; no longer U6.3 (Q0), U7.15 (Reset)
- net at U6.1 (Q5): now also U2.1 (X4); no longer U2.12 (X3)
- net at U6.10 (Q4): now also U2.12 (X3); no longer U2.15 (X2)
- net at U5.1, U6.11 (Q9), U6.13 (CKEN): no longer U2.4 (X7)
- net at U6.2 (Q1): now also U2.13 (X0)
- net at U6.4 (Q2): now also U2.14 (X1); no longer U2.13 (X0)
- net at U6.5 (Q6): now also U2.5 (X5); no longer U2.1 (X4)
- net at U6.6 (Q7): now also U2.2 (X6); no longer U2.5 (X5)
- net at U6.7 (Q3): now also U2.15 (X2); no longer U2.14 (X1)
- net at U6.9 (Q8): now also U2.4 (X7); no longer U2.2 (X6)
- net at U7.1 (Q5): now also U3.1 (X4); no longer U3.5 (X5)
- net at U7.10 (Q4): now also U3.12 (X3); no longer U3.1 (X4)
- net at U7.11 (Q9): now also D3.2 (A)
- net at U7.2 (Q1): now also U3.13 (X0); no longer U3.14 (X1)
- net at U7.3 (Q0): no longer U3.13 (X0)
- net at U7.4 (Q2): now also U3.14 (X1); no longer U3.15 (X2)
- net at U7.5 (Q6): now also U3.5 (X5); no longer U3.2 (X6)
- net at U7.6 (Q7): now also U3.2 (X6); no longer U3.4 (X7)
- net at U7.7 (Q3): now also U3.15 (X2); no longer U3.12 (X3)
- net at U7.9 (Q8): now also U3.4 (X7); no longer D3.2 (A)
- net at U12.11 (Q9), U12.13 (CKEN), U9.4 (X7): now also U5.8; no longer U5.5
- net at U13.14 (CLK): now also U5.10; no longer U5.4
- new net: U6.3 (Q0), U7.15 (Reset), U?.6
Other:
- moved on the sheet: J2, U3, U6

Commit message: ffs routing done
Parts:
- added C5: 10uf, Capacitor_THT:CP_Radial_D8.0mm_P2.50mm, symbol Device:CP
- added C6, C7: 224nf, Capacitor_THT:C_Disc_D4.3mm_W1.9mm_P5.00mm, symbol Device:C
- added U11: 40106, Package_DIP:DIP-16_W7.62mm_Socket, symbol 4xxx_IEEE:40106
- added unit 4 of U5
- C4: value 22uf -> 10uf
- D2, D3, D5, D6: value D -> 1N4148
- TP6: value TestPoint -> -12V
- U5: renamed from U?; footprint (none) -> Package_DIP:DIP-14_W7.62mm_Socket
Connections:
- net FreqMulOut is gone; now on net FreqMultOut: U4.4 (FOUT)
- net Vdd is gone; now on net +12V: U1.16 (Vdd), U1.16 (Vdd), U8.16 (Vdd), U8.16 (Vdd)
- net Vss is gone; now on net GND: U1.8 (Vss), U1.8 (Vss), U8.8 (Vss), U8.8 (Vss)
- net CP1: no longer U8.1 (CP), U8.9 (CP)
- net FreqDivOut: now also U11.6; no longer U12.3 (Q0), U13.15 (Reset)
- net FreqMultOut: now also U5.12
- net GND: now also J2.9 (Pin_9), C5.2, C6.2, C7.1
- net SigIn: now also U11.1, U11.4; no longer U4.14 (SigIn), U5.4
- net at U1.10 (Q4), U2.6 (Inh): now also U1.15 (D)
- net at R2.1, R3.1, U4.9 (VCOin): now also C5.1
- net at U12.1 (Q5): now also U9.1 (X4); no longer U9.12 (X3)
- net at U12.10 (Q4): now also U9.12 (X3); no longer U9.15 (X2)
- net at U12.11 (Q9), U12.13 (CKEN), U5.8: no longer U9.4 (X7)
- net at U12.2 (Q1): now also U9.13 (X0)
- net at U12.4 (Q2): now also U9.14 (X1); no longer U9.13 (X0)
- net at U12.5 (Q6): now also U9.5 (X5); no longer U9.1 (X4)
- net at U12.6 (Q7): now also U9.2 (X6); no longer U9.5 (X5)
- net at U12.7 (Q3): now also U9.15 (X2); no longer U9.14 (X1)
- net at U12.9 (Q8): now also U9.4 (X7); no longer U9.2 (X6)
- net at U8.10 (Q4), U9.6 (Inh): now also U8.15 (D)
- net at U13.1 (Q5): now also U10.1 (X4); no longer U10.5 (X5)
- net at U13.10 (Q4): now also U10.12 (X3); no longer U10.1 (X4)
- net at U13.11 (Q9): now also D6.2 (A)
- net at U13.2 (Q1): now also U10.13 (X0); no longer U10.14 (X1)
- net at U13.3 (Q0): no longer U10.13 (X0)
- net at U13.4 (Q2): now also U10.14 (X1); no longer U10.15 (X2)
- net at U13.5 (Q6): now also U10.5 (X5); no longer U10.2 (X6)
- net at U13.6 (Q7): now also U10.2 (X6); no longer U10.4 (X7)
- net at U13.7 (Q3): now also U10.15 (X2); no longer U10.12 (X3)
- net at U13.9 (Q8): now also U10.4 (X7); no longer D6.2 (A)
- net D1A renamed CP2
- net CP2: now also U8.1 (CP), U8.9 (CP); no longer U1.7 (D)
- net D1B renamed MR
- net MR: now also U1.14 (MR), U1.6 (MR), U8.14 (MR), U8.6 (MR); no longer U1.15 (D)
- net D2A renamed D2
- removed net D2B: J2.9 (Pin_9), U8.15 (D)
- removed net MR1: J2.5 (Pin_5), U1.14 (MR), U1.6 (MR), U8.14 (MR), U8.6 (MR)
- new net: C6.1, U11.3, U5.4
- new net: C7.2, U11.5, U5.11
- new net: U11.2, U4.14 (SigIn)
- new net: U12.3 (Q0), U13.15 (Reset), U5.13
- new net D1: J2.5 (Pin_5), U1.7 (D)
Other:
- moved on the sheet: C1, C2, C4, D1, D3, D4, D5, D6, J1, J2, R2, R3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

Commit message: added bypass caps
Parts:
- added C10, C11, C12, C13, C14, C15, C16, C18, C19, C20, C21, C8, C9: 10nf, Capacitor_SMD:C_1206_3216Metric_Pad1.42x1.75mm_HandSolder, symbol Device:C_Small
- added unit 7 of U11
- U11: symbol 4xxx_IEEE:40106 -> 4xxx:40106
Connections:
- net +12V: now also C10.2, C11.2, C12.2, C13.2, C14.2, C15.2, C16.2, C18.2, C19.2, C20.2, C21.2, C8.2, C9.2, U11.14 (VDD)
- net GND: now also C10.1, C11.1, C12.1, C13.1, C14.1, C15.1, C16.1, C18.1, C19.1, C20.1, C21.1, C8.1, C9.1, U11.7 (VSS)
Other:
- moved on the sheet: U5E
